File: Hardware/WandStrobeDriver/WandStrobeDriver.kicad_sch (KiCad schematic)
At the start: 28 parts, among them J1 12V IN, J2 MARKER A (origin), J3 MARKER B, J4 MARKER C (+X), J5 MARKER D (+Y), Q1 DMP3098L-7, SW1 POWER, U1 TLC555CP

Commit message: Strobe driver rev B: 9 V, fixed resistors, and the driver PCB
Rev A ran 12 V and put a constant-current sink on every marker board. The
sink cost 1.6 V of headroom - a Vbe of sense, a Vce of regulation, and the
input Schottky - and that 1.6 V was the entire reason 12 V was needed. What
it bought was marker-to-marker matching of about 5%, against ~3% run-to-run
repeatability in the characterisation itself. It was buying matching finer
than the measurement can resolve, so it is gone.

The marker board is now the board that was already characterised plus a
connector: four LEDs, one ballast resistor, eight parts. The existing bench
markers plug straight into the driver, and at 9 V they draw 36 mA - the
characterised operating point - so the strobe test is directly comparable
with the DC rows in LED_characterisation.xlsx.

Also settled from the datasheet (Kingbright L-7113SF7C, DSAB9772):

- 1.6 V is the forward drop AT 20 mA, not a constant. At 36 mA it is ~1.48 V,
  so the string is 5.9 V rather than the 6.4 V a flat 1.6 V implies. The
  workbook's 38.2 mA was computed from the 1.6 V figure; the real current
  through 68 R at 9 V is nearer 43 mA. Worth measuring, it appears in the
  thesis.
- The 1 A peak rating is quoted at a 10 us pulse, 80x shorter than ours, so
  it does not apply. What does apply is average power: 0.19 mW against an
  80 mW limit.
- The 20 degree viewing angle is the ring artefact, which is why the emitters
  must be aimed tangentially rather than radially.

No diode across R2, and none is needed. The usual sub-50% duty trick assumes
the LEDs are on when OUT is high; they are not. Q1 is P-channel on the high
side and conducts when OUT is low, so the short state is already the one we
want. Adding the diode would force R1 small and sink ~20 mA through DISCH for
the whole 327 ms off-time, against the 9 uA the circuit actually draws.

Driver PCB: 80 x 60 mm, two layers, 0 DRC violations, 0 unconnected pads.
B.Cu is the ground return; only the gate esc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
Parts:
- removed RV1: 1M RATE, Potentiometer_THT:Potentiometer_Bourns_3296W_Vertical, symbol Device:R_Potentiometer_Trim
- removed RV2: 2k WIDTH, Potentiometer_THT:Potentiometer_Bourns_3296W_Vertical, symbol Device:R_Potentiometer_Trim
- C1: value 1000u/25V -> 1000u/16V
- F1: value 1A -> 500mA
- J1: value 12V IN -> 9V IN
- R1: value 470k -> 1M; footprint Resistor_SMD:R_0805_2012Metric -> Resistor_THT:R_Axial_DIN0207_L6.3mm_D2.5mm_P10.16mm_Horizontal
- R2: value 470 -> 3k6; footprint Resistor_SMD:R_0805_2012Metric -> Resistor_THT:R_Axial_DIN0207_L6.3mm_D2.5mm_P10.16mm_Horizontal
- R5: value 10k -> 22k
- SW1: footprint Button_Switch_THT:SW_CK_JS202011AQN_DPDT_Angled -> Button_Switch_THT:SW_Slide_SPDT_Angled_CK_OS102011MA1Q; symbol Switch:SW_SPST -> Switch:SW_SPDT
Connections:
- net at R1.2: now also R2.1, U1.7 (DISCH)
- net at C6.1, U1.2 (TRIG), U1.6 (THRES): now also R2.2
- net at J1.1 (Pin_1): now also SW1.2 (B); no longer SW1.1 (A)
- net at F1.1: now also SW1.1 (A); no longer SW1.2 (B)
- net +12V renamed +9V
- no-connect marks 0 -> 1
Other:
- note added: "Q1 sees Vgs = -9 V, so a +/-12 V part (AO3401A) is now legal too. DMP3098L-7 is +/-20 V and costs the same. Do not fit a +/-8 V part."
- note added: "Regime B (long camera exposure, short flash). The flash - not the shutter - defines the instant, so every camera whose shutter is open records the same ~1 ms. One timer for the whole wand, so "dark" always means occluded and never out of phase. NO DIODE ACROSS R2, AND NONE IS NEEDED. The usual trick for sub-50% duty assumes the LEDs are on when OUT is HIGH. They are not: Q1 is P-channel on the hi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"
- note added: "STROBE DRIVER rev B - one timer, nothing to adjust"
- note removed: "Q1 must be rated Vgs +/-20 V: the gate swings the full 12 V rail. Common SOT-23 P-FETs (AO3401A, Si2301) are only +/-8..12 V - do not fit one."
- note removed: "Regime B (long camera exposure, short flash). The flash - not the shutter - defines the instant, so every camera whose shutter is open sees the same 300 us. Duty ~0.09%, so pulsed overdrive is available. TIMING plain astable, no diode. R1+RV1 >> R2+RV2 puts the SHORT state on OUT LOW, and Q1 (P-channel, high side) conducts when OUT is low. The diode-across-R2 trick is NOT used: it would burn Vcc/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"
- note removed: "STROBE DRIVER - one timer for the whole wand"
- title: Wand strobe driver - TLC555 + high-side P-FET, 12 V -> Wand strobe driver - TLC555 + high-side P-FET, 9 V
- moved on the sheet: C6, J1
