File: Hardware/WandStrobeBreadboard/WandStrobeBreadboard.kicad_sch (KiCad schematic)
At the start: 26 parts, among them J1 9V IN, J2 MARKER A (origin), J3 MARKER B, J4 MARKER C (+X), J5 MARKER D (+Y), Q1 DMP3098L-7, SW1 POWER, U1 TLC555CP

Commit message: Add the N-channel breadboard schematic as a real, ERC-checked sheet
WandStrobeBreadboard is the bench build for a lab with only N-channel parts.
Drawing it in KiCad rather than by hand means ERC and the netlist verify the
one thing that is easy to get wrong: the diode across R2 sits anode on the
DISCH node and cathode on THRES/TRIG, so the charge path bypasses R2 and the
discharge path does not.

Differences from the PCB, and nothing else changes:

  R1  1M   -> 3k3     charge path, now the short state
  R2  3k3  -> 1M      discharge path, now the long state
  D3       -> 1N4148  across R2, anode at DISCH
  Q1  P-ch high side -> IRF540N N-ch low side
  R4  100k pull-up to source -> 10k pull-down to ground

Marker pin 1 is now permanently on +9V and pin 2 is the switched return, so
the marker positives are live whenever the board is powered. That is the
safety property the high-side PCB keeps and this variant gives up.

Timing is unchanged: 1075 us, 3.06 Hz, 0.33 % duty.
Parts:
- removed Q1: DMP3098L-7, Package_TO_SOT_SMD:SOT-23, symbol Transistor_FET:Q_PMOS_GSD
- added D3: 1N4148, Diode_THT:D_DO-35_SOD27_P10.16mm_Horizontal, symbol Device:D
- added Q1: IRF540N, Package_TO_SOT_THT:TO-220-3_Vertical, symbol Transistor_FET:Q_NMOS_GSD
- C2, C4, C5: footprint Capacitor_SMD:C_0805_2012Metric -> Capacitor_THT:C_Disc_D5.0mm_W2.5mm_P5.00mm
- D1: value SS34 -> 1N5817; footprint Diode_SMD:D_SMA -> Diode_THT:D_DO-41_SOD81_P10.16mm_Horizontal
- D2: footprint LED_SMD:LED_0805_2012Metric -> Diode_THT:D_DO-41_SOD81_P10.16mm_Horizontal
- R1: value 1M -> 3k3
- R10, R3, R5: footprint Resistor_SMD:R_0805_2012Metric -> Resistor_THT:R_Axial_DIN0207_L6.3mm_D2.5mm_P10.16mm_Horizontal
- R2: value 3k3 -> 1M
- R4: value 100k -> 10k; footprint Resistor_SMD:R_0805_2012Metric -> Resistor_THT:R_Axial_DIN0207_L6.3mm_D2.5mm_P10.16mm_Horizontal
- TP1: value GATE -> OUT
- TP2: value SW_LED -> LED_RTN
Connections:
- net +9V: now also J2.1 (Pin_1), J3.1 (Pin_1), J4.1 (Pin_1), J5.1 (Pin_1); no longer R4.1
- net GND: now also R4.2, Q1.2 (S); no longer J2.2 (Pin_2), J3.2 (Pin_2), J4.2 (Pin_2), J5.2 (Pin_2)
- net at R3.2: now also R4.1, Q1.1 (G); no longer R4.2
- net at C6.1, R2.2, U1.2 (TRIG)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: now also D3.1 (K)
- net at R1.2, R2.1, U1.7 (DISCH): now also D3.2 (A)
- net GATE: no longer names the net of R3.1, TP1.1, U1.3 (OUT)
- removed net SW_LED: J2.1 (Pin_1), J3.1 (Pin_1), J4.1 (Pin_1), J5.1 (Pin_1), TP2.1
- new net LED_RTN: J2.2 (Pin_2), J3.2 (Pin_2), J4.2 (Pin_2), J5.2 (Pin_2), Q1.3 (D), TP2.1
Other:
- note removed: "Q1 sees Vgs = -9 V, so a +/-12 V part (AO3401A) is now legal too. DMP3098L-7 is +/-20 V and costs the same. Do not fit a +/-8 V part."
- note removed: "Regime B (long camera exposure, short flash). The flash - not the shutter - defines the instant, so every camera whose shutter is open records the same ~1 ms. One timer for the whole wand, so "dark" always means occluded and never out of phase. NO DIODE ACROSS R2, AND NONE IS NEEDED. The usual trick for sub-50% duty assumes the LEDs are on when OUT is HIGH. They are not: Q1 is P-channel on the hi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"
- note removed: "STROBE DRIVER rev B - one timer, nothing to adjust"
- title: Wand strobe driver - TLC555 + high-side P-FET, 9 V -> Wand strobe driver - BREADBOARD variant, N-channel low side, 9 V
